Commit message: Automated update by GitHub Action

File: description/robot.urdf (robot description, URDF)
Before this commit: robot servobot, 13 links, 12 joints
Joints:
- joint BL_BotLeg: origin xyz=7.35523e-16 0.112 -4.16334e-17 rpy=-3.14159 2.22045e-16 1.5708 -> xyz=7.49401e-16 0.112 -5.55112e-17 rpy=-3.14159 -1.25634e-16 1.5708
- joint BL_Hip: origin xyz=-2.77556e-16 -8.67362e-18 -0.16305 rpy=-2.95937e-15 4.82972e-15 1.76636e-15 -> xyz=-3.46945e-17 7.97973e-17 -0.16305 rpy=-2.6263e-15 4.2217e-15 4.73371e-15
- joint BL_TopLeg: origin xyz=-0.02225 0.028265 -0.02 rpy=2.55043e-16 1.5708 0 -> xyz=-0.02225 0.028265 -0.02 rpy=2.18733e-17 1.5708 0
- joint BR_BotLeg: origin xyz=-2.77556e-17 0.112 4.16334e-17 rpy=3.14159 -8.49659e-15 1.5708 -> xyz=-8.32667e-17 0.112 2.77556e-17 rpy=3.14159 -7.48348e-15 1.5708
- joint BR_Hip: origin xyz=0.1103 1.42247e-16 -0.16305 rpy=2.95937e-15 -2.70816e-15 -3.14159 -> xyz=0.1103 6.43582e-16 -0.16305 rpy=2.90386e-15 -2.93515e-15 -3.14159
- joint FL_BotLeg: origin xyz=4.16334e-17 0.112 -1.34615e-15 rpy=3.14159 1.42113e-14 1.5708 -> xyz=2.77556e-17 0.112 -1.33227e-15 rpy=3.14159 1.42668e-14 1.5708
- joint FL_Hip: origin xyz=-0.0551412 0.0821676 -0.0155485 rpy=-1.5708 -1.5886e-15 2.70816e-15 -> xyz=0.0563298 -0.0818149 -0.0155485 rpy=-1.5708 -5.23321e-15 -3.14159
- joint FL_TopLeg: origin xyz=-0.0773912 0.102168 -0.0438135 rpy=-1.5708 6.02296e-15 -1.5708 -> xyz=0.0785798 -0.101815 -0.0438135 rpy=-1.5708 1.50479e-14 1.5708
- joint FR_BotLeg: origin xyz=-8.32667e-17 0.112 4.57967e-16 rpy=-3.14159 -8.68483e-15 1.5708 -> xyz=-8.32667e-17 0.112 4.71845e-16 rpy=-3.14159 -8.68483e-15 1.5708
- joint FR_Hip: origin xyz=0.1103 1.49186e-16 -3.33067e-16 rpy=-3.14159 -2.71489e-15 -3.14159 -> xyz=0.1103 5.6205e-16 -2.77556e-16 rpy=-3.14159 -2.65351e-15 -3.14159
- joint FR_TopLeg: origin xyz=-0.02225 0.028265 -0.02 rpy=-1.66533e-16 1.5708 0 -> xyz=-0.02225 0.028265 -0.02 rpy=-1.04424e-16 1.5708 0
