Commit message: Automated update by GitHub Action

File: urdf/servobot.urdf (robot description, URDF)
Before this commit: robot servobot, 9 links, 8 joints
Joints:
- joint bl_hip: limit effort=10 velocity=10 -> lower=-1 upper=1 effort=10 velocity=10; type fixed -> revolute
- joint bl_top: limit effort=10 velocity=10 -> lower=-3.14159 upper=3.14159 effort=10 velocity=10; type fixed -> revolute
- joint br_hip: limit effort=10 velocity=10 -> lower=-1 upper=1 effort=10 velocity=10; type fixed -> revolute
- joint br_top: limit effort=10 velocity=10 -> lower=-3.14159 upper=3.14159 effort=10 velocity=10; type fixed -> revolute
- joint fl_hip: limit effort=10 velocity=10 -> lower=-1 upper=1 effort=10 velocity=10; type fixed -> revolute
- joint fl_top: limit effort=10 velocity=10 -> lower=-3.14159 upper=3.14159 effort=10 velocity=10; type fixed -> revolute
- joint fr_hip: limit effort=10 velocity=10 -> lower=-1 upper=1 effort=10 velocity=10; type fixed -> revolute
- joint fr_top: limit effort=10 velocity=10 -> lower=-3.14159 upper=3.14159 effort=10 velocity=10; type fixed -> revolute

Commit message: Automated update by GitHub Action

File: urdf/servobot.urdf (robot description, URDF)
Before this commit: robot servobot, 9 links, 8 joints
Links:
- removed link legasm
- removed link legasm2
- removed link legasmflipped
- removed link legasmflipped2
- added link 2000_0025_0002, mass 0.0170887; collision mesh filename=package://servobot_description/meshes/2000_0025_0002.stl; collision mesh filename=package://servobot_description/meshes/mg995_gear2.stl
- added link 2000_0025_0002_2, mass 0.0170887; collision mesh filename=package://servobot_description/meshes/2000_0025_0002.stl; collision mesh filename=package://servobot_description/meshes/mg995_gear2.stl
- added link 2000_0025_0002_3, mass 0.0170887; collision mesh filename=package://servobot_description/meshes/2000_0025_0002.stl; collision mesh filename=package://servobot_description/meshes/mg995_gear2.stl
- added link 2000_0025_0002_4, mass 0.0170887; collision mesh filename=package://servobot_description/meshes/2000_0025_0002.stl; collision mesh filename=package://servobot_description/meshes/mg995_gear2.stl
- added link part_1, mass 0.0738028; collision mesh filename=package://servobot_description/meshes/2000_0025_0002__2.stl; collision mesh filename=package://servobot_description/meshes/mg995_gear2.stl
- added link part_1_2, mass 0.0738028; collision mesh filename=package://servobot_description/meshes/2000_0025_0002__2.stl; collision mesh filename=package://servobot_description/meshes/mg995_gear2.stl
- added link part_1_3, mass 0.0738028; collision mesh filename=package://servobot_description/meshes/2000_0025_0002__2.stl; collision mesh filename=package://servobot_description/meshes/mg995_gear2.stl
- added link part_1_4, mass 0.0738028; collision mesh filename=package://servobot_description/meshes/2000_0025_0002__2.stl; collision mesh filename=package://servobot_description/meshes/mg995_gear2.stl
Joints:
- added joint bl_bot: type revolute, parent part_1, child 2000_0025_0002, origin xyz=4.16334e-17 0.0851134 0.0159 rpy=3.14159 2.00394e-17 -1.5708, axis 0 0 1, limit lower=-3.14159 upper=3.14159 effort=10 velocity=10
- added joint br_bot: type revolute, parent part_1_4, child 2000_0025_0002_4, origin xyz=-2.77556e-17 0.0851134 0.0159 rpy=-3.14159 -1.22783e-16 1.5708, axis 0 0 1, limit lower=-3.14159 upper=3.14159 effort=10 velocity=10
- added joint fl_bot: type revolute, parent part_1_2, child 2000_0025_0002_2, origin xyz=4.16334e-17 0.0851134 0.0159 rpy=3.14159 -0 -1.5708, axis 0 0 1, limit lower=-3.14159 upper=3.14159 effort=10 velocity=10
- added joint fr_bot: type revolute, parent part_1_3, child 2000_0025_0002_3, origin xyz=-2.63678e-16 0.0851134 0.0159 rpy=-3.14159 6.20402e-16 1.5708, axis 0 0 1, limit lower=-3.14159 upper=3.14159 effort=10 velocity=10
- joint bl_top: child legasm2 -> part_1
- joint br_top: child legasmflipped2 -> part_1_4
- joint fl_top: child legasm -> part_1_2
- joint fr_top: child legasmflipped -> part_1_3

Commit message: Automated update by GitHub Action

File: urdf/servobot.urdf (robot description, URDF)
Before this commit: robot servobot, 13 links, 12 joints
Joints:
- joint bl_bot: limit lower=-3.14159 upper=3.14159 effort=10 velocity=10 -> lower=-1.5708 upper=1.5708 effort=10 velocity=10
- joint bl_top: limit lower=-3.14159 upper=3.14159 effort=10 velocity=10 -> lower=-1.5708 upper=1.5708 effort=10 velocity=10
- joint br_bot: limit lower=-3.14159 upper=3.14159 effort=10 velocity=10 -> lower=-1.5708 upper=1.5708 effort=10 velocity=10
- joint br_top: limit lower=-3.14159 upper=3.14159 effort=10 velocity=10 -> lower=-1.5708 upper=1.5708 effort=10 velocity=10
- joint fl_bot: limit lower=-3.14159 upper=3.14159 effort=10 velocity=10 -> lower=-1.5708 upper=1.5708 effort=10 velocity=10
- joint fl_top: limit lower=-3.14159 upper=3.14159 effort=10 velocity=10 -> lower=-1.5708 upper=1.5708 effort=10 velocity=10
- joint fr_bot: limit lower=-3.14159 upper=3.14159 effort=10 velocity=10 -> lower=-1.5708 upper=1.5708 effort=10 velocity=10
- joint fr_top: limit lower=-3.14159 upper=3.14159 effort=10 velocity=10 -> lower=-1.5708 upper=1.5708 effort=10 velocity=10
