Commit message: Automated update by GitHub Action

File: urdf/robot.urdf (robot description, URDF)
Before this commit: robot servobot, 13 links, 12 joints
Joints:
- joint bl_bot: limit lower=-1.5708 upper=1.5708 effort=10 velocity=10 -> lower=-1.5708 upper=1.5708 effort=1.8 velocity=6
- joint bl_hip: limit lower=-1 upper=1 effort=10 velocity=10 -> lower=-1 upper=1 effort=1.8 velocity=6
- joint bl_top: limit lower=-1.5708 upper=1.5708 effort=10 velocity=10 -> lower=-1.5708 upper=1.5708 effort=1.8 velocity=6
- joint br_bot: limit lower=-1.5708 upper=1.5708 effort=10 velocity=10 -> lower=-1.5708 upper=1.5708 effort=1.8 velocity=6
- joint br_hip: limit lower=-1 upper=1 effort=10 velocity=10 -> lower=-1 upper=1 effort=1.8 velocity=6
- joint br_top: limit lower=-1.5708 upper=1.5708 effort=10 velocity=10 -> lower=-1.5708 upper=1.5708 effort=1.8 velocity=6
- joint fl_bot: limit lower=-1.5708 upper=1.5708 effort=10 velocity=10 -> lower=-1.5708 upper=1.5708 effort=1.8 velocity=6
- joint fl_hip: limit lower=-1 upper=1 effort=10 velocity=10 -> lower=-1 upper=1 effort=1.8 velocity=6
- joint fl_top: limit lower=-1.5708 upper=1.5708 effort=10 velocity=10 -> lower=-1.5708 upper=1.5708 effort=1.8 velocity=6
- joint fr_bot: limit lower=-1.5708 upper=1.5708 effort=10 velocity=10 -> lower=-1.5708 upper=1.5708 effort=1.8 velocity=6
- joint fr_hip: limit lower=-1 upper=1 effort=10 velocity=10 -> lower=-1 upper=1 effort=1.8 velocity=6
- joint fr_top: limit lower=-1.5708 upper=1.5708 effort=10 velocity=10 -> lower=-1.5708 upper=1.5708 effort=1.8 velocity=6

Commit message: Automated update by GitHub Action

File: urdf/robot.urdf (robot description, URDF)
Before this commit: robot servobot, 13 links, 12 joints
Links:
- link chassisasm: mass 1.41284 -> 1.00595

Commit message: Automated update by GitHub Action

File: urdf/robot.urdf (robot description, URDF)
Before this commit: robot servobot, 13 links, 12 joints
Joints:
- joint bl_hip: limit lower=-1 upper=1 effort=1.8 velocity=6 -> lower=-0.00913852 upper=0.00913852 effort=1.8 velocity=6
- joint br_hip: limit lower=-1 upper=1 effort=1.8 velocity=6 -> lower=-0.00913852 upper=0.00913852 effort=1.8 velocity=6
- joint fl_hip: limit lower=-1 upper=1 effort=1.8 velocity=6 -> lower=-0.00913852 upper=0.00913852 effort=1.8 velocity=6
- joint fr_hip: limit lower=-1 upper=1 effort=1.8 velocity=6 -> lower=-0.00913852 upper=0.00913852 effort=1.8 velocity=6

Commit message: Automated update by GitHub Action

File: urdf/robot.urdf (robot description, URDF)
Before this commit: robot servobot, 13 links, 12 joints
Joints:
- joint bl_bot: limit lower=-1.5708 upper=1.5708 effort=1.8 velocity=6 -> lower=-1.5708 upper=1.5708 effort=2.1 velocity=6.5
- joint bl_hip: limit lower=-0.00913852 upper=0.00913852 effort=1.8 velocity=6 -> lower=-0.00913852 upper=0.00913852 effort=2.1 velocity=6.5
- joint bl_top: limit lower=-1.5708 upper=1.5708 effort=1.8 velocity=6 -> lower=-1.5708 upper=1.5708 effort=2.1 velocity=6.5
- joint br_bot: limit lower=-1.5708 upper=1.5708 effort=1.8 velocity=6 -> lower=-1.5708 upper=1.5708 effort=2.1 velocity=6.5
- joint br_hip: limit lower=-0.00913852 upper=0.00913852 effort=1.8 velocity=6 -> lower=-0.00913852 upper=0.00913852 effort=2.1 velocity=6.5
- joint br_top: limit lower=-1.5708 upper=1.5708 effort=1.8 velocity=6 -> lower=-1.5708 upper=1.5708 effort=2.1 velocity=6.5
- joint fl_bot: limit lower=-1.5708 upper=1.5708 effort=1.8 velocity=6 -> lower=-1.5708 upper=1.5708 effort=2.1 velocity=6.5
- joint fl_hip: limit lower=-0.00913852 upper=0.00913852 effort=1.8 velocity=6 -> lower=-0.00913852 upper=0.00913852 effort=2.1 velocity=6.5
- joint fl_top: limit lower=-1.5708 upper=1.5708 effort=1.8 velocity=6 -> lower=-1.5708 upper=1.5708 effort=2.1 velocity=6.5
- joint fr_bot: limit lower=-1.5708 upper=1.5708 effort=1.8 velocity=6 -> lower=-1.5708 upper=1.5708 effort=2.1 velocity=6.5
- joint fr_hip: limit lower=-0.00913852 upper=0.00913852 effort=1.8 velocity=6 -> lower=-0.00913852 upper=0.00913852 effort=2.1 velocity=6.5
- joint fr_top: limit lower=-1.5708 upper=1.5708 effort=1.8 velocity=6 -> lower=-1.5708 upper=1.5708 effort=2.1 velocity=6.5

Commit message: Automated update by GitHub Action

File: urdf/robot.urdf (robot description, URDF)
Before this commit: robot servobot, 13 links, 12 joints
Joints:
- joint bl_hip: limit lower=-0.00913852 upper=0.00913852 effort=2.1 velocity=6.5 -> lower=-0.523599 upper=0.523599 effort=2.1 velocity=6.5
- joint br_hip: limit lower=-0.00913852 upper=0.00913852 effort=2.1 velocity=6.5 -> lower=-0.523599 upper=0.523599 effort=2.1 velocity=6.5
- joint fl_hip: limit lower=-0.00913852 upper=0.00913852 effort=2.1 velocity=6.5 -> lower=-0.523599 upper=0.523599 effort=2.1 velocity=6.5
- joint fr_hip: limit lower=-0.00913852 upper=0.00913852 effort=2.1 velocity=6.5 -> lower=-0.523599 upper=0.523599 effort=2.1 velocity=6.5
